File: GrapeNano.sch (KiCad schematic (older format))
At the start: 31 parts, among them P1 USB_OTG, P2 ICSP, SW1 SW_Push, U1 LM1117-5.0, U2 CH340G, U3 ATMEGA328P-AU, Y1 12MHz, Y2 16Mhz

Commit message: CH340G cambiado por CH340C
Parts:
- removed U2: CH340G, Housings_SOIC:SOIC-16_3.9x9.9mm_Pitch1.27mm, symbol CH340G_D-SUN-V3.0-cache:CH340G
- removed Y1: 12MHz, Clocks:RESONATOR-SMD-3.2X1.3, symbol device:Resonator_Small
- added U2: CH340C, Package_SO:SOIC-16_3.9x9.9mm_P1.27mm, symbol ch340:CH340C
- A1: symbol modules:Arduino_Nano_v3.x -> GrapeNano-rescue:Arduino_Nano_v3.x-modules
- C1, C2, C4, C5, C6, C8, C9: symbol device:C_Small -> GrapeNano-rescue:C_Small-device
- C3, C7: symbol device:CP_Small -> GrapeNano-rescue:CP_Small-device
- D1, D2: symbol device:D_Small_ALT -> GrapeNano-rescue:D_Small_ALT-device
- D3: symbol device:D_Schottky_Small -> GrapeNano-rescue:D_Schottky_Small-device
- D4, D5: symbol device:LED_Small -> GrapeNano-rescue:LED_Small-device
- F1: symbol device:Polyfuse_Small -> GrapeNano-rescue:Polyfuse_Small-device
- P1: symbol conn:USB_OTG -> GrapeNano-rescue:USB_OTG-conn
- P2: symbol conn:CONN_02X03 -> GrapeNano-rescue:CONN_02X03-conn
- R1, R2, R3, R4, R5, R6, R7: symbol device:R_Small -> GrapeNano-rescue:R_Small-device
- SW1: symbol switches:SW_Push -> GrapeNano-rescue:SW_Push-switches
- U1: symbol regul:LM1117-5.0 -> GrapeNano-rescue:LM1117-5.0-regul
- U3: symbol atmel:ATMEGA328P-AU -> GrapeNano-rescue:ATMEGA328P-AU-atmel
- Y2: symbol device:Resonator_Small -> GrapeNano-rescue:Resonator_Small-device
Connections:
- net +3V3: now also C1.1
- net +5V: now also C6.1, C7.1, C9.1, U3.18 (AVCC), U3.4 (VCC), U3.6 (VCC), U2.16 (VCC); no longer C1.1
- net DTR: now also U2.13 (DTR)
- net GND: now also U2.1 (GND)
- net at P1.2 (D-): now also U2.6 (UD-)
- net at P1.3 (D+): now also U2.5 (UD+)
- net at R3.2: now also U2.2 (TXD)
- net at R4.2: now also U2.3 (RXD)
- net at C1.2: now also U2.4 (V3)
- no-connect marks 7 -> 9
Other:
- moved on the sheet: C2, P2, U1
