File: GrapeNano.sch (KiCad schematic (older format))
At the start: 1 part

Commit message: Haciendo el esquema
Parts:
- added C?: C, symbol device:C
- added C?: CP, symbol device:CP
- added C?: 100n, symbol device:C_Small
- added D?: LED_Small, symbol device:LED_Small
- added D?: GREEN, symbol device:D_Small_ALT
- added D?: RED, symbol device:D_Small_ALT
- added F?: 500mA, symbol device:Polyfuse_Small
- added P?: USB_OTG, symbol conn:USB_OTG
- added R? (x2): 10k, symbol device:R_Small
- added R? (x2): 1k, symbol device:R_Small
- added SW?: SW_Push, symbol switches:SW_Push
- added U?: LM1117-5.0, symbol GrapeNano-rescue:LM1117-5.0
- added U?: CH340G, SOIC-16_N, symbol CH340G_D-SUN-V3.0-cache:CH340G
- added Y?: Resonator_Small, symbol device:Resonator_Small
- added Y?: 12MHz, symbol device:Resonator_Small
- U?: symbol ATMEGA328P-AU -> atmel:ATMEGA328P-AU
Connections:
- net labels added: +3.3V, +5V, GND, RX, TX, VUSB
- wire segments 0 -> 47
- no-connect marks 0 -> 4

Commit message: Esquema terminado
Parts:
- removed C?: C, symbol device:C
- removed C?: CP, symbol device:CP
- removed U?: LM1117-5.0, symbol GrapeNano-rescue:LM1117-5.0
- added 1u, C? (x2): 100n, symbol device:C_Small
- added A?: Arduino_Nano_v3.x, Modules:Arduino_Nano, symbol modules:Arduino_Nano_v3.x
- added C?: 1u, symbol device:C_Small
- added C?: 4.7u, symbol device:CP_Small
- added C?: 1uF, symbol device:C_Small
- added D?: BAT20J, symbol device:D_Schottky_Small
- added P?: ICSP, symbol conn:CONN_02X03
- added R? (x2): 1k, symbol device:R_Small
- added U?: LM1117-5.0, symbol regul:LM1117-5.0
- D?: value LED_Small -> LED_PWD
- Y?: value Resonator_Small -> 16Mhz
Connections:
- net labels added: A0, A1, A2, A3, A4, A5, A6, A7, AREF, D0, D0-RX, D1, D1-TX, D10, D11, D11-MOSI, D12, D12-MISO, D13, D13-SCK, D2, D3, D4, D5, D6, D7, D8, D9, DTR, RESET, VIN
- net labels removed: RX, TX
- wire segments 47 -> 165
- no-connect marks 4 -> 7
Other:
- moved on the sheet: C?, D?, F?, P?, R?, SW?, U?, Y?

Commit message: Componentes colocados y comenzando a enrutar
Parts:
- added C3: 4.7u, Capacitors_Tantalum_SMD:CP_Tantalum_Case-A_EIA-3216-18_Reflow, symbol device:CP_Small
- added C4: 100n, Capacitors_SMD:C_0603, symbol device:C_Small
- added D5: LED_13, LEDs:LED_0805, symbol device:LED_Small
- added R7: 1k, Resistors_SMD:R_0603, symbol device:R_Small
- A1: renamed from A?; footprint Modules:Arduino_Nano -> Modules:Arduino_Nano_WithMountingHoles
- C1, C2, C5, C6, C8: renamed from C?; footprint (none) -> Capacitors_SMD:C_0603
- C7: renamed from C?; footprint (none) -> Capacitors_Tantalum_SMD:CP_Tantalum_Case-A_EIA-3216-18_Reflow
- C9: renamed from 1u; footprint (none) -> Capacitors_SMD:C_0603
- D1, D2, D4: renamed from D?; footprint (none) -> LEDs:LED_0805
- D3: renamed from D?; footprint (none) -> Diodes_SMD:D_SOD-323
- F1: renamed from F?; footprint (none) -> Capacitors_SMD:C_0603_HandSoldering
- P1: renamed from P?; footprint (none) -> Connectors_USB:USB_Micro-B_Molex-105017-0001
- P2: renamed from P?; footprint (none) -> Connectors:2X3
- R1, R2, R3, R4, R5, R6: renamed from R?; footprint (none) -> Resistors_SMD:R_0603
- SW1: renamed from SW?; footprint (none) -> Buttons_Switches_SMD:SW_SPST_B3U-1000P
- U1: renamed from U?; footprint (none) -> TO_SOT_Packages_SMD:SOT-223
- U2: renamed from U?; footprint SOIC-16_N -> Housings_SOIC:SOIC-16_3.9x9.9mm_Pitch1.27mm
- U3: renamed from U?; footprint TQFP32 -> Housings_QFP:TQFP-32_7x7mm_Pitch0.8mm
- Y1, Y2: renamed from Y?; footprint (none) -> Clocks:RESONATOR-SMD-3.2X1.3
Connections:
- net D0 is gone; now on net D0-RX: A1.2 (D0/RX)
- net D1 is gone; now on net D1-TX: A1.1 (D1/TX)
- net D11 is gone; now on net D11-MOSI: A1.14 (D11)
- net D12 is gone; now on net D12-MISO: A1.15 (D12)
- net D13 is gone; now on net D13-SCK: A1.16 (D13)
- net D13-SCK: now also R7.1
- net GND: now also C3.2, C4.2, D5.1 (K)
- net VUSB: now also C3.1, C4.1
- new net: D5.2 (A), R7.2

Commit message: mandado a fabrica
Parts:
- removed U2: CH340G, Housings_SOIC:SOIC-16_3.9x9.9mm_Pitch1.27mm, symbol CH340G_D-SUN-V3.0-cache:CH340G
- removed Y1: 12MHz, Clocks:RESONATOR-SMD-3.2X1.3, symbol device:Resonator_Small
- added U2: CH340C, Housings_SOIC:SOIC-16_3.9x9.9mm_Pitch1.27mm, symbol ch340:CH340C
Connections:
- net +3V3: now also C1.1
- net +5V: now also U2.16 (VCC); no longer C1.1
- net DTR: now also U2.13 (DTR)
- net GND: now also C1.2, U2.1 (GND), U2.4 (V3)
- net at P1.2 (D-): now also U2.6 (UD-)
- net at P1.3 (D+): now also U2.5 (UD+)
- net at R3.2: now also U2.2 (TXD)
- net at R4.2: now also U2.3 (RXD)
- no-connect marks 7 -> 9
Other:
- moved on the sheet: C5
Changed lines of the file:
@@
 EESchema Schematic File Version 4
 LIBS:GrapeNano-cache
-EELAYER 26 0
+EELAYER 29 0
 EELAYER END
 $Descr A4 11693 8268
@@
 	0    -1   1    0
 $EndComp
-$Comp
-L CH340G_D-SUN-V3.0-cache:CH340G U2
-U 1 1 5C72806C
-P 3300 4150
-F 0 "U2" H 3300 4837 60  0000 C CNN
-F 1 "CH340G" H 3300 4731 60  0000 C CNN
-F 2 "Housings_SOIC:SOIC-16_3.9x9.9mm_Pitch1.27mm" H 3300 3600 40  0001 C CNN
-F 3 "" H 3300 4150 60  0000 C CNN
-	1    3300 4150
-	1    0    0    -1
-$EndComp
 Wire Wire Line
 	2000 4150 2250 4150
@@
 	2050 4450 2050 4700
 NoConn ~ 2000 4350
-$Comp
-L device:Resonator_Small Y1
-U 1 1 5C73E2E6
-P 2400 4600
-F 0 "Y1" H 2525 4675 50  0000 L CNN
-F 1 "12MHz" H 2525 4600 50  0000 L CNN
-F 2 "Clocks:RESONATOR-SMD-3.2X1.3" H 2375 4600 50  0001 C CNN
-F 3 "" H 2375 4600 50  0001 C CNN
-	1    2400 4600
-	1    0    0    -1
-$EndComp
-Wire Wire Line
-	2500 4500 2500 4450
-Wire Wire Line
-	2500 4450 2600 4450
-Wire Wire Line
-	2600 4350 2300 4350
-Wire Wire Line
-	2300 4350 2300 4500
-$Comp
-L power:GND #PWR0105
-U 1 1 5C73E6B1
-P 2400 4850
-F 0 "#PWR0105" H 2400 4600 50  0001 C CNN
-F 1 "GND" H 2400 4700 50  0000 C CNN
-F 2 "" H 2400 4850 50  0001 C CNN
-F 3 "" H 2400 4850 50  0001 C CNN
-	1    2400 4850
-	1    0    0    -1
-$EndComp
-Wire Wire Line
-	2400 4800 2400 4850
 $Comp
 L power:GND #PWR0106
@@
 	2600 3850 2400 3850
 Wire Wire Line
-	2600 4050 2100 4050
+	2600 4050 2450 4050
 Wire Wire Line
 	2100 4050 2100 3800
@@
 	1    0    0    -1
 $EndComp
-$Comp
-L power:+5V #PWR0107
-U 1 1 5C73F57A
-P 2100 3500
-F 0 "#PWR0107" H 2100 3350 50  0001 C CNN
-F 1 "+5V" H 2100 3640 50  0000 C CNN
-F 2 "" H 2100 3500 50  0001 C CNN
-F 3 "" H 2100 3500 50  0001 C CNN
-	1    2100 3500
-	1    0    0    -1
-$EndComp
 Wire Wire Line
 	2100 3500 2100 3600
@@
 L power:+5V #PWR0108
 U 1 1 5C73FA2E
-P 4150 3500
-F 0 "#PWR0108" H 4150 3350 50  0001 C CNN
-F 1 "+5V" H 4150 3640 50  0000 C CNN
-F 2 "" H 4150 3500 50  0001 C CNN
-F 3 "" H 4150 3500 50  0001 C CNN
-	1    4150 3500
-	1    0    0    -1
-$EndComp
-Wire Wire Line
-	4150 3500 4150 3750
-Wire Wire Line
-	4150 3750 4000 3750
-NoConn ~ 4000 3850
-NoConn ~ 4000 4250
-NoConn ~ 4000 4150
+P 3450 3500
+F 0 "#PWR0108" H 3450 3350 50  0001 C CNN
+F 1 "+5V" H 3450 3640 50  0000 C CNN
+F 2 "" H 3450 3500 50  0001 C CNN
+F 3 "" H 3450 3500 50  0001 C CNN
+	1    3450 3500
+	1    0    0    -1
+$EndComp
+Wire Wire Line
+	3450 3500 3450 3750
+Wire Wire Line
+	3450 3750 3300 3750
+NoConn ~ 3300 3850
+NoConn ~ 3300 4250
+NoConn ~ 3300 4150
 $Comp
 L device:Polyfuse_Small F1
@@
 L device:C_Small C5
 U 1 1 5C74BF6B
-P 4400 4050
-F 0 "C5" H 4600 4050 50  0000 R CNN
-F 1 "100n" H 4650 4150 50  0000 R CNN
-F 2 "Capacitors_SMD:C_0603" H 4400 4050 50  0001 C CNN
-F 3 "" H 4400 4050 50  0001 C CNN
-	1    4400 4050
-	1    0    0    -1
-$EndComp
-Text GLabel 4400 3850 1    39   Input ~ 0
+P 3700 4050
+F 0 "C5" H 3900 4050 50  0000 R CNN
+F 1 "100n" H 3950 4150 50  0000 R CNN
+F 2 "Capacitors_SMD:C_0603" H 3700 4050 50  0001 C CNN
+F 3 "" H 3700 4050 50  0001 C CNN
+	1    3700 4050
+	1    0    0    -1
+$EndComp
+Text GLabel 3700 3850 1    39   Input ~ 0
 DTR
-Text GLabel 4400 4250 3    39   Input ~ 0
+Text GLabel 3700 4250 3    39   Input ~ 0
 RESET
 Wire Wire Line
-	4400 3850 4400 3950
-Wire Wire Line
-	4400 4150 4400 4250
-Text GLabel 4050 4050 2    39   Input ~ 0
+	3700 3850 3700 3950
+Wire Wire Line
+	3700 4150 3700 4250
+Text GLabel 3350 4050 2    39   Input ~ 0
 DTR
 Wire Wire Line
-	4000 4050 4050 4050
-NoConn ~ 4000 3950
-NoConn ~ 4000 4350
-NoConn ~ 4000 4450
+	3300 4050 3350 4050
+NoConn ~ 3300 3950
+NoConn ~ 3300 4350
+NoConn ~ 3300 4450
 $Comp
 L power:GND #PWR0111
@@
 Text GLabel 9450 3150 0    39   Input ~ 0
 D1-TX
+$Comp
+L ch340:CH340C U2
+U 1 1 5CC4D035
+P 2950 4050
+F 0 "U2" H 2950 4575 50  0000 C CNN
+F 1 "CH340C" H 2950 4484 50  0000 C CNN
+F 2 "Housings_SOIC:SOIC-16_3.9x9.9mm_Pitch1.27mm" H 2850 4200 50  0001 C CNN
+F 3 "" H 2850 4200 50  0001 C CNN
+	1    2950 4050
+	1    0    0    -1
+$EndComp
+NoConn ~ 2600 4350
+NoConn ~ 2600 4450
+$Comp
+L power:+3.3V #PWR?
+U 1 1 5CC7CA92
+P 2100 3500
+F 0 "#PWR?" H 2100 3350 50  0001 C CNN
+F 1 "+3.3V" H 2100 3640 50  0000 C CNN
+F 2 "" H 2100 3500 50  0001 C CNN
+F 3 "" H 2100 3500 50  0001 C CNN
+	1    2100 3500
+	1    0    0    -1
+$EndComp
+$Comp
+L power:GND #PWR?
+U 1 1 5CC805C4
+P 2450 4700
+F 0 "#PWR?" H 2450 4450 50  0001 C CNN
+F 1 "GND" H 2450 4550 50  0000 C CNN
+F 2 "" H 2450 4700 50  0001 C CNN
+F 3 "" H 2450 4700 50  0001 C CNN
+	1    2450 4700
+	1    0    0    -1
+$EndComp
+Wire Wire Line
+	2450 4050 2450 4700
+Connection ~ 2450 4050
+Wire Wire Line
+	2450 4050 2100 4050
 $EndSCHEMATC

Commit message: Errores corregidos y mandado a fábrica
Corto en el condensador C1 y U3 sin alimentación
Parts:
- A1: symbol modules:Arduino_Nano_v3.x -> GrapeNano-rescue:Arduino_Nano_v3.x-modules
- C1, C2, C4, C5, C6, C8, C9: symbol device:C_Small -> GrapeNano-rescue:C_Small-device
- C3, C7: symbol device:CP_Small -> GrapeNano-rescue:CP_Small-device
- D1, D2: symbol device:D_Small_ALT -> GrapeNano-rescue:D_Small_ALT-device
- D3: symbol device:D_Schottky_Small -> GrapeNano-rescue:D_Schottky_Small-device
- D4, D5: symbol device:LED_Small -> GrapeNano-rescue:LED_Small-device
- F1: symbol device:Polyfuse_Small -> GrapeNano-rescue:Polyfuse_Small-device
- P1: symbol conn:USB_OTG -> GrapeNano-rescue:USB_OTG-conn
- P2: symbol conn:CONN_02X03 -> GrapeNano-rescue:CONN_02X03-conn
- R1, R2, R3, R4, R5, R6, R7: symbol device:R_Small -> GrapeNano-rescue:R_Small-device
- SW1: symbol switches:SW_Push -> GrapeNano-rescue:SW_Push-switches
- U1: symbol regul:LM1117-5.0 -> GrapeNano-rescue:LM1117-5.0-regul
- U3: symbol atmel:ATMEGA328P-AU -> GrapeNano-rescue:ATMEGA328P-AU-atmel
- Y2: symbol device:Resonator_Small -> GrapeNano-rescue:Resonator_Small-device
Connections:
- net +3V3: now also C1.2, U2.4 (V3); no longer C1.1
- net +5V: now also C6.1, C7.1, C9.1, U3.18 (AVCC), U3.4 (VCC), U3.6 (VCC)
- net GND: now also C1.1; no longer C1.2, U2.4 (V3)
Changed lines of the file:
@@
 $EndDescr
 $Comp
-L atmel:ATMEGA328P-AU U3
+L GrapeNano-rescue:ATMEGA328P-AU-atmel U3
 U 1 1 588F3A7E
 P 6700 3500
@@
 $EndComp
 $Comp
-L device:Resonator_Small Y2
+L GrapeNano-rescue:Resonator_Small-device Y2
 U 1 1 589903E4
 P 8500 3050
@@
 $EndComp
 $Comp
-L switches:SW_Push SW1
+L GrapeNano-rescue:SW_Push-switches SW1
 U 1 1 58990510
 P 5200 4350
@@
 $EndComp
 $Comp
-L device:LED_Small D4
+L GrapeNano-rescue:LED_Small-device D4
 U 1 1 589905E7
 P 8500 4800
@@
 $EndComp
 $Comp
-L device:D_Small_ALT D1
+L GrapeNano-rescue:D_Small_ALT-device D1
 U 1 1 5899073E
 P 1800 2900
@@
 $EndComp
 $Comp
-L conn:USB_OTG P1
+L GrapeNano-rescue:USB_OTG-conn P1
 U 1 1 589907F1
 P 1700 4250
@@
 	2600 3850 2400 3850
 Wire Wire Line
-	2600 4050 2450 4050
-Wire Wire Line
 	2100 4050 2100 3800
 $Comp
-L device:C_Small C1
+L GrapeNano-rescue:C_Small-device C1
 U 1 1 5C73F321
 P 2100 3700
@@
 NoConn ~ 3300 4150
 $Comp
-L device:Polyfuse_Small F1
+L GrapeNano-rescue:Polyfuse_Small-device F1
 U 1 1 5C7403D0
 P 1900 3700
@@
 	2450 3950 2600 3950
 $Comp
-L device:D_Small_ALT D2
+L GrapeNano-rescue:D_Small_ALT-device D2
 U 1 1 5C742B81
 P 1800 3050
@@
 $EndComp
 $Comp
-L device:R_Small R2
+L GrapeNano-rescue:R_Small-device R2
 U 1 1 5C743231
 P 1500 3050
@@
 $EndComp
 $Comp
-L device:R_Small R1
+L GrapeNano-rescue:R_Small-device R1
 U 1 1 5C74332C
 P 1500 2900
@@
 	1600 2900 1700 2900
 $Comp
-L device:R_Small R3
+L GrapeNano-rescue:R_Small-device R3
 U 1 1 5C744BC1
 P 2350 3150
@@
 $EndComp
 $Comp
-L device:R_Small R4
+L GrapeNano-rescue:R_Small-device R4
 U 1 1 5C744C4F
 P 2500 3150
@@
 	1900 3050 2200 3050
 $Comp
-L device:C_Small C5
+L GrapeNano-rescue:C_Small-device C5
 U 1 1 5C74BF6B
 P 3700 4050
@@
 	8700 3050 8750 3050
 $Comp
-L device:C_Small C9
+L GrapeNano-rescue:C_Small-device C9
 U 1 1 5C755AC1
 P 5500 2500
@@
 $EndComp
 $Comp
-L device:C_Small C6
+L GrapeNano-rescue:C_Small-device C6
 U 1 1 5C755DCD
 P 5100 2500
@@
 Connection ~ 5100 2600
 $Comp
-L device:C_Small C8
+L GrapeNano-rescue:C_Small-device C8
 U 1 1 5C75FAE9
 P 5650 3150
@@
 AREF
 $Comp
-L modules:Arduino_Nano_v3.x A1
+L GrapeNano-rescue:Arduino_Nano_v3.x-modules A1
 U 1 1 5C763F92
 P 10050 3650
@@
 	9950 2600 9950 2650
 $Comp
-L device:CP_Small C7
+L GrapeNano-rescue:CP_Small-device C7
 U 1 1 5C780A63
 P 5300 2500
@@
 Connection ~ 5200 4100
 $Comp
-L device:R_Small R5
+L GrapeNano-rescue:R_Small-device R5
 U 1 1 5C78C554
 P 5200 3950
@@
 RESET
 $Comp
-L conn:CONN_02X03 P2
+L GrapeNano-rescue:CONN_02X03-conn P2
 U 1 1 5C7A0CE0
 P 4450 5700
@@
 	4200 5800 4100 5800
 $Comp
-L device:R_Small R6
+L GrapeNano-rescue:R_Small-device R6
 U 1 1 5C7C0006
 P 8500 4500
@@
 	7700 4100 7800 4100
 $Comp
-L regul:LM1117-5.0 U1
+L GrapeNano-rescue:LM1117-5.0-regul U1
 U 1 1 5C86D8DE
 P 2400 5650
@@
 	2400 5950 2400 6000
 $Comp
-L device:C_Small C2
+L GrapeNano-rescue:C_Small-device C2
 U 1 1 5C87B1F2
 P 2800 5800
@@
 $EndComp
 $Comp
-L device:D_Schottky_Small D3
+L GrapeNano-rescue:D_Schottky_Small-device D3
 U 1 1 5C89014E
 P 6700 5700
@@
 	7000 5700 7000 5500
 $Comp
-L device:CP_Small C3
+L GrapeNano-rescue:CP_Small-device C3
 U 1 1 5C89F877
 P 3100 2800
@@
 $EndComp
 $Comp
-L device:C_Small C4
+L GrapeNano-rescue:C_Small-device C4
 U 1 1 5C89F8F5
 P 3350 2800
@@
 	7850 2900 7850 2200
 $Comp
-L device:LED_Small D5
+L GrapeNano-rescue:LED_Small-device D5
 U 1 1 5C8BFD6E
 P 7850 1800
@@
 $EndComp
 $Comp
-L device:R_Small R7
+L GrapeNano-rescue:R_Small-device R7
 U 1 1 5C8BFD75
 P 7850 2100
@@
 NoConn ~ 2600 4450
 $Comp
-L power:+3.3V #PWR?
-U 1 1 5CC7CA92
+L power:+5V #PWR?
+U 1 1 5D0E9B6F
+P 5100 2300
+F 0 "#PWR?" H 5100 2150 50  0001 C CNN
+F 1 "+5V" H 5100 2440 50  0000 C CNN
+F 2 "" H 5100 2300 50  0001 C CNN
+F 3 "" H 5100 2300 50  0001 C CNN
+	1    5100 2300
+	1    0    0    -1
+$EndComp
+Wire Wire Line
+	5100 2300 5100 2400
+Connection ~ 5100 2400
+Wire Wire Line
+	2100 4050 2250 4050
+$Comp
+L power:GND #PWR?
+U 1 1 5D0F376E
 P 2100 3500
-F 0 "#PWR?" H 2100 3350 50  0001 C CNN
-F 1 "+3.3V" H 2100 3640 50  0000 C CNN
+F 0 "#PWR?" H 2100 3250 50  0001 C CNN
+F 1 "GND" H 2100 3350 50  0000 C CNN
 F 2 "" H 2100 3500 50  0001 C CNN
 F 3 "" H 2100 3500 50  0001 C CNN
 	1    2100 3500
-	1    0    0    -1
-$EndComp
-$Comp
-L power:GND #PWR?
-U 1 1 5CC805C4
-P 2450 4700
-F 0 "#PWR?" H 2450 4450 50  0001 C CNN
-F 1 "GND" H 2450 4550 50  0000 C CNN
-F 2 "" H 2450 4700 50  0001 C CNN
-F 3 "" H 2450 4700 50  0001 C CNN
-	1    2450 4700
-	1    0    0    -1
-$EndComp
-Wire Wire Line
-	2450 4050 2450 4700
-Connection ~ 2450 4050
-Wire Wire Line
-	2450 4050 2100 4050
+	-1   0    0    1
+$EndComp
+$Comp
+L power:+3.3V #PWR?
+U 1 1 5D0F4074
+P 2250 4000
+F 0 "#PWR?" H 2250 3850 50  0001 C CNN
+F 1 "+3.3V" H 2250 4140 50  0000 C CNN
+F 2 "" H 2250 4000 50  0001 C CNN
+F 3 "" H 2250 4000 50  0001 C CNN
+	1    2250 4000
+	1    0    0    -1
+$EndComp
+Wire Wire Line
+	2250 4000 2250 4050
+Connection ~ 2250 4050
+Wire Wire Line
+	2250 4050 2600 4050
 $EndSCHEMATC
