File: GrapeNano.kicad_pcb (KiCad board)
At the start: 2 copper layers, 18.5 x 43.7 mm, 33 parts, among them P1 USB_OTG, P2 ICSP, SW1 SW_Push, U1 LM1117-5.0, U2 CH340G, U3 ATMEGA328P-AU, Y1 12MHz, Y2 16Mhz

Commit message: mandado a fabrica
Parts:
- removed Y1: 12MHz, Clocks:RESONATOR-SMD-3.2X1.3
- U2: value CH340G -> CH340C
- moved P1 0.10 mm to (157.4, 121.0)
Connections:
- C1 pad 1: +5V -> +3V3
- C1 pad 2: Net-(C1-Pad2) -> GND
- U2 pad 4: Net-(C1-Pad2) -> GND
Routing:
- net +3V3: track 0.00 -> 33.1 mm, vias 0 -> 1
- net Net-(C1-Pad2): track 8.29 -> 0.00 mm
- net Net-(U2-Pad7): track 5.51 -> 0.00 mm
- net GND: track 46.2 -> 51.4 mm
- net Net-(U2-Pad8): track 2.76 -> 0.00 mm
- net A6: track 22.1 -> 23.0 mm
- net Net-(P1-Pad2): track 16.5 -> 17.3 mm
- net +5V: track 79.2 -> 78.6 mm
- net AREF: track 7.71 -> 8.37 mm
